File: DarkQuest_SiPM_Motherboard.kicad_pcb (KiCad board)
At the start: 2 copper layers, 100 x 100 mm, 38 parts, among them J1 Conn_Coaxial, J10 Conn_Coaxial, J11 Conn_Coaxial, J12 Conn_Coaxial, J13 8-102202-4, J14 8-102202-4, J15 8-102202-4, J16 8-102202-4, J2 Conn_Coaxial, J21 RJ45_Shielded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

Commit message: Added HDMI option
Parts:
- removed J24: SiPM Header, RJJS-88-122-E7V-022:chip_carrier_pin_header
- removed SW1, SW2, SW3, SW4: SW_Push_DPDT, Relay_SMD:Nidec_DPDT_CS422YTA
- added C1: 10nF 100V, Capacitor_SMD:C_1206_3216Metric_Pad1.33x1.80mm_HandSolder, F.Cu at (-19.4, 66.5)
- added C2: 10nF 100V, Capacitor_SMD:C_1206_3216Metric_Pad1.33x1.80mm_HandSolder, F.Cu at (-19.4, 99.4)
- added C3: 10nF 100V, Capacitor_SMD:C_1206_3216Metric_Pad1.33x1.80mm_HandSolder, F.Cu at (10.3, 66.5)
- added C4: 10nF 100V, Capacitor_SMD:C_1206_3216Metric_Pad1.33x1.80mm_HandSolder, F.Cu at (10.3, 99.4)
- added J3: SiPM Header, RJJS-88-122-E7V-022:chip_carrier_pin_header, F.Cu at (-8.66, 51.0)
- added J4: SiPM Header, RJJS-88-122-E7V-022:chip_carrier_pin_header, F.Cu at (-8.66, 84.0)
- added J5: SiPM Header, RJJS-88-122-E7V-022:chip_carrier_pin_header, F.Cu at (21.0, 51.0)
- added J6: SiPM Header, RJJS-88-122-E7V-022:chip_carrier_pin_header, F.Cu at (127.8, 72.4)
- added JP1: SolderJumper_2_Open, Jumper:SolderJumper-2_P1.3mm_Open_RoundedPad1.0x1.5mm, B.Cu at (26.6, 82.5)
- added JP2: SolderJumper_2_Open, Jumper:SolderJumper-2_P1.3mm_Open_RoundedPad1.0x1.5mm, B.Cu at (43.0, 77.0)
- added JP3: SolderJumper_2_Open, Jumper:SolderJumper-2_P1.3mm_Open_RoundedPad1.0x1.5mm, B.Cu at (26.6, 88.0)
- added JP4: SolderJumper_2_Open, Jumper:SolderJumper-2_P1.3mm_Open_RoundedPad1.0x1.5mm, B.Cu at (33.0, 88.0)
- renumbered J21 to J2
Connections:
- J2 pad 1: /K1 -> /K0
- J2 pad 2: /A1 -> /A0
- J2 pad 3: /K2 -> /K1
- J2 pad 4: /A3 -> /A2
- J2 pad 5: /K3 -> /K2
- J2 pad 6: /A2 -> /A1
- J2 pad 7: /K4 -> /K3
- J2 pad 8: /A4 -> /A3
- J2 pad SH: Net-(JP1-B) -> GND
Routing:
- net (no net): track 0.00 -> 22.3 mm
- net /SiPM Support 3/A_PreAtten: track 0.00 -> 7.70 mm
- net /A3_PreAtten: track 7.70 -> 0.00 mm
- net Net-(SW4-A-Pad3): track 5.58 -> 0.00 mm
- net Net-(SW2-A-Pad3): track 5.58 -> 0.00 mm
- net Net-(SW1-A-Pad3): track 5.58 -> 0.00 mm
- net Net-(SW3-A-Pad3): track 5.58 -> 0.00 mm
- net GND: track 0.00 -> 0.52 mm
- net Net-(JP1-B): track 230.4 -> 229.9 mm
- removed copper zone on B.Cu, net GND1
- removed copper zone on B.Cu, net GND3
- removed copper zone on B.Cu, net GND4
