File: DarkQuest_SiPM_Motherboard.kicad_pcb (KiCad board)
At the start: 2 copper layers, 100 x 100 mm, 38 parts, among them J1 Conn_Coaxial, J10 Conn_Coaxial, J11 Conn_Coaxial, J12 Conn_Coaxial, J13 8-102202-4, J14 8-102202-4, J15 8-102202-4, J16 8-102202-4, J2 Conn_Coaxial, J21 RJ45_Shielded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

Commit message: Finished initial routing
Parts:
- removed the J1 at (138.3, 144.7)
- removed J10, J11, J12, J9: Conn_Coaxial, Connector_Coaxial:WR-MMCX_Wuerth_66012102111404_Vertical
- removed J13, J14, J15, J16: 8-102202-4, Connector_PinHeader_2.54mm:PinHeader_1x03_P2.54mm_Vertical
- removed the J2 at (117.0, 55.8)
- removed the J3 at (138.0, 55.8)
- removed the J4 at (61.5, 55.8)
- removed JP1, JP2, JP3, JP4: SolderJumper_2_Open, Jumper:SolderJumper-2_P1.3mm_Open_RoundedPad1.0x1.5mm
- removed SW1, SW2, SW3, SW4: SW_Push_DPDT, Relay_SMD:Nidec_DPDT_CS422YTA
- removed U1, U2, U3, U4: ~, Resistor_SMD:D10AA20Z4
- moved C2 9.71 mm to (79.7, 127.5), turned to 90 degrees
- moved C3 8.86 mm to (135.2, 72.1), turned to 90 degrees
- moved C4 8.84 mm to (79.8, 72.1), turned to 90 degrees
- moved C1 8.76 mm to (135.1, 127.5), turned to 90 degrees
- renumbered J21 to J1, J23 to J2, J22 to J3, J24 to J4, J25 to J5
Connections:
- C1 pad 1: GND1 -> /K0
- C1 pad 2: /K1 -> GND
- C2 pad 1: GND2 -> /K1
- C2 pad 2: /K2 -> GND
- C3 pad 1: GND3 -> /K2
- C3 pad 2: /K3 -> GND
- C4 pad 1: GND4 -> /K3
- C4 pad 2: /K4 -> GND
- J1 pad 1: /K1 -> /K0
- J1 pad 2: /A1 -> /A0
- J1 pad 3: /K2 -> /K1
- J1 pad 4: /A3 -> /A2
- J1 pad 5: /K3 -> /K2
- J1 pad 6: /A2 -> /A1
- J1 pad 7: /K4 -> /K3
- J1 pad 8: /A4 -> /A3
- J1 pad SH: Net-(JP1-B) -> GND
- J2 pad 1: /A1_PreAtten -> /A0
- J2 pad 2: GND1 -> GND
- J2 pad 3: /K1 -> /K0
- J3 pad 1: /A2_PreAtten -> /A1
- J3 pad 2: GND2 -> GND
- J3 pad 3: /K2 -> /K1
- J4 pad 1: /A3_PreAtten -> /A2
- J4 pad 2: GND3 -> GND
- J4 pad 3: /K3 -> /K2
- J5 pad 1: /A4_PreAtten -> /A3
- J5 pad 2: GND4 -> GND
- J5 pad 3: /K4 -> /K3
Routing:
- net Net-(JP1-B): track 230.4 -> 0.00 mm
- net /A4: track 106.7 -> 0.00 mm
- net /K4: track 87.1 -> 0.00 mm
- net /K1: track 86.9 -> 26.8 mm
- net GND1: track 55.6 -> 0.00 mm, vias 2 -> 0
- net /K0: track 0.00 -> 54.3 mm
- net /K3: track 98.0 -> 61.6 mm
- net GND3: track 29.2 -> 0.00 mm, vias 1 -> 0
- net GND4: track 28.2 -> 0.00 mm, vias 1 -> 0
- net /A2: track 77.8 -> 50.2 mm
- net /A3: track 95.1 -> 68.7 mm
- net GND2: track 25.7 -> 0.00 mm, vias 1 -> 0
- net /A1: track 60.8 -> 81.9 mm
- net Net-(SW4-0): track 13.6 -> 0.00 mm, vias 1 -> 0
- net /A0: track 0.00 -> 13.5 mm
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- added copper zone on B.Cu, net GND
- removed copper zone on B.Cu, net GND1
- removed copper zone on B.Cu, net GND2
- removed copper zone on B.Cu, net GND3
- removed copper zone on B.Cu, net GND4
